File: MarlinOctoHat/MarlinOctoHat.kicad_sch (KiCad schematic)
At the start: 29 parts, among them J1 Screw_Terminal_01x03, J2 Conn_01x02_Male, J3 Conn_01x04_Male, J4 Conn_01x03_Male, J5 Conn_01x04_Male, J6 Conn_01x02_Male, J7 Conn_01x04_Male, J8 Conn_01x07_Female, Q1 BC547, Q2 BC547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

Commit message: Update MarlinOctoHat.kicad_sch
Other:
- note added: "OLED : SSD1306 / SSD1309 / SSH1106 (SPI mode) LCD : ST7920 (RepRapDiscount Full Graphic Smart Controller)"
- note removed: "OLED : SSD1306 / SSD1309 / SSH1106 (SPI mode) LCD : ST7920 (*NOT IMPLEMENTTD* RepRapDiscount Full Graphic Smart Controller)"
Changed lines of the file:
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@@
     (effects (font (size 1.27 1.27)) (justify left bottom))
   )
-  (text "OLED : SSD1306 / SSD1309 / SSH1106 (SPI mode)\nLCD : ST7920 (*NOT IMPLEMENTTD* RepRapDiscount Full Graphic Smart Controller)"
+  (text "OLED : SSD1306 / SSD1309 / SSH1106 (SPI mode)\nLCD : ST7920 (RepRapDiscount Full Graphic Smart Controller)"
     (at 26.67 121.92 0)
     (effects (font (size 1.27 1.27)) (justify left bottom))
